Commit message: Second commit

File: my_robot/urdf/my_robot.xacro (robot description, xacro)
@@ -1,49 +1,22 @@
+<?xml version='1.0'?>
 <robot name="my_robot" xmlns:xacro="http://www.ros.org/wiki/xacro">
   <xacro:include filename="$(find my_robot)/urdf/my_robot.gazebo" />
-  <link name="robot_footprint"></link>
-  <gazebo reference="left_wheel">
-    <material>Gazebo/Green</material>
-  </gazebo>
-  <gazebo reference="right_wheel">
-    <material>Gazebo/Green</material>
-  </gazebo>
-  <gazebo reference="camera">
-    <material>Gazebo/Gray</material>
-  </gazebo>
   <gazebo reference="chassis">
     <material>Gazebo/Orange</material>
   </gazebo>
+  <gazebo reference="left_wheel">
+    <material>Gazebo/Gray</material>
+  </gazebo>
+  <gazebo reference="right_wheel">
+    <material>Gazebo/Gray</material>
+  </gazebo>
+  <gazebo reference="camera">
+    <material>Gazebo/PurpleGlow</material>
+  </gazebo>
+  <link name="robot_footprint"></link>
   <joint name="robot_footprint_joint" type="fixed">
     <origin xyz="0 0 0" rpy="0 0 0" />
     <parent link="robot_footprint" />
     <child link="chassis" />
-  </joint>
-  <joint type="continuous" name="left_wheel_hinge">
-    <origin xyz="0 0.3 0" rpy="0 0 0" />
-    <child link="left_wheel" />
-    <parent link="chassis" />
-    <axis xyz="0 1 0" rpy="0 0 0" />
-    <limit effort="10000" velocity="1000" />
-    <dynamics damping="1.0" friction="1.0" />
-  </joint>
-  <joint type="continuous" name="right_wheel_hinge">
-    <origin xyz="0 -0.3 0" rpy="0 0 0" />
-    <child link="right_wheel" />
-    <parent link="chassis" />
-    <axis xyz="0 1 0" rpy="0 0 0" />
-    <limit effort="10000" velocity="1000" />
-    <dynamics damping="1.0" friction="1.0" />
-  </joint>
-  <joint type="fixed" name="camera_joint">
-    <origin xyz="0.25 0 0" rpy="0 0 0" />
-    <child link="camera" />
-    <parent link="chassis" />
-    <axis xyz="0 1 0" />
-  </joint>
-  <joint type="fixed" name="hokuyo_joint">
-    <origin xyz="0.15 0 0.1" rpy="0 0 0" />
-    <child link="hokuyo" />
-    <parent link="chassis" />
-    <axis xyz="0 1 0" />
   </joint>
   <link name='chassis'>
@@ -61,5 +34,5 @@
       <origin xyz="0 0 0" rpy=" 0 0 0" />
       <geometry>
-        <box size=".5 .5 .1" />
+        <box size=".4 .3 .1" />
       </geometry>
     </collision>
@@ -67,5 +40,5 @@
       <origin xyz="0 0 0" rpy=" 0 0 0" />
       <geometry>
-        <box size=".5 .5 .1" />
+        <box size=".4 .3 .1" />
       </geometry>
     </visual>
@@ -95,12 +68,11 @@
     </visual>
   </link>
-  <link name="right_wheel">
+  <link name="left_wheel">
     <inertial>
+      <origin xyz="0 0 0" rpy="0 1.5707 1.5707" />
       <mass value="5" />
-      <origin xyz="0 0 0" rpy="0 1.5707 1.5707" />
       <inertia
-        ixx="0.1" ixy="0.0" ixz="0.0"
-        iyy="0.1" iyz="0.0"
-        izz="0.1"
+        ixx="0.1" ixy="0" ixz="0"
+        iyy="0.1" iyz="0" izz="0.1"
       />
     </inertial>
@@ -108,5 +80,5 @@
       <origin xyz="0 0 0" rpy="0 1.5707 1.5707" />
       <geometry>
-        <cylinder radius="0.105" length="0.05" />
+        <cylinder radius="0.1" length="0.05" />
       </geometry>
     </collision>
@@ -114,16 +86,15 @@
       <origin xyz="0 0 0" rpy="0 1.5707 1.5707" />
       <geometry>
-        <cylinder radius="0.105" length="0.05" />
+        <cylinder radius="0.1" length="0.05" />
       </geometry>
     </visual>
   </link>
-  <link name="left_wheel">
+  <link name="right_wheel">
     <inertial>
+      <origin xyz="0 0 0" rpy="0 1.5707 1.5707" />
       <mass value="5" />
-      <origin xyz="0 0 0" rpy="0 1.5707 1.5707" />
       <inertia
-        ixx="0.1" ixy="0.0" ixz="0.0"
-        iyy="0.1" iyz="0.0"
-        izz="0.1"
+        ixx="0.1" ixy="0" ixz="0"
+        iyy="0.1" iyz="0" izz="0.1"
       />
     </inertial>
@@ -131,5 +102,5 @@
       <origin xyz="0 0 0" rpy="0 1.5707 1.5707" />
       <geometry>
-        <cylinder radius="0.105" length="0.05" />
+        <cylinder radius="0.1" length="0.05" />
       </geometry>
     </collision>
@@ -137,49 +108,65 @@
       <origin xyz="0 0 0" rpy="0 1.5707 1.5707" />
       <geometry>
-        <cylinder radius="0.105" length="0.05" />
+        <cylinder radius="0.1" length="0.05" />
       </geometry>
     </visual>
   </link>
+  <joint name="left_wheel_hinge" type="continuous">
+    <origin xyz="0 0.225 0" rpy="0 0 0" />
+    <child link="left_wheel" />
+    <parent link="chassis" />
+    <axis xyz="0 1 0" rpy="0 0 0" />
+    <limit effort="10000" velocity="1000" />
+    <dynamics damping="1.0" friction="1.0" />
+  </joint>
+  <joint name="right_wheel_hinge" type="continuous">
+    <origin xyz="0 -0.225 0" rpy="0 0 0" />
+    <child link="right_wheel" />
+    <parent link="chassis" />
+    <axis xyz="0 1 0" rpy="0 0 0" />
+    <limit effort="10000" velocity="1000" />
+    <dynamics damping="1.0" friction="1.0" />
+  </joint>
   <link name="camera">
+    <origin xyz="0 0 0" rpy="0 0 0" />
     <inertial>
       <mass value="0.1" />
-      <origin xyz="0 0 0" rpy="0 0 0" />
       <inertia
         ixx="1e-6" ixy="0" ixz="0"
-        iyy="1e-6" iyz="0"
-        izz="1e-6"
+        iyy="1e-6" iyz="0" izz="1e-6"
       />
     </inertial>
     <collision>
-      <origin xyz="0 0 0" rpy="0 0 0" />
       <geometry>
-        <box size="0.1 0.05 0.05" />
+        <box size="0.05 0.05 0.05" />
       </geometry>
     </collision>
     <visual>
-      <origin xyz="0 0 0" rpy="0 0 0" />
       <geometry>
-        <box size="0.1 0.05 0.05" />
+        <box size="0.05 0.05 0.05" />
       </geometry>
     </visual>
   </link>
+  <joint name="camera_joint" type="fixed">
+    <axis xyz="0 1 0" />
+    <origin xyz="0.2 0 0" rpy="0 0 0" />
+    <parent link="chassis" />
+    <child link="camera" />
+  </joint>
   <link name="hokuyo">
+    <origin xyz="0 0 0" rpy="0 0 0" />
     <inertial>
       <mass value="1e-5" />
-      <origin xyz="0 0 0" rpy="0 0 0" />
       <inertia
         ixx="1e-6" ixy="0" ixz="0"
-        iyy="1e-6" iyz="0"
-        izz="1e-6"
+        iyy="1e-6" iyz="0" izz="1e-6"
       />
     </inertial>
     <collision>
-      <origin xyz="0 0 0" rpy="0 0 0" />
       <geometry>
-        <box size="0.1 0.1 0.1" />
+        <box size=".1 .1 .1" />
       </geometry>
     </collision>
     <visual>
-      <origin xyz="0 0 0" rpy="0 0 0" />
       <geometry>
         <mesh filename="package://my_robot/meshes/hokuyo.dae" />
@@ -187,3 +174,9 @@
     </visual>
   </link>
+  <joint name="hokuyo_joint" type="fixed">
+    <axis xyz="0 1 0" />
+    <origin xyz="0.15 0 0.1" rpy="0 0 0" />
+    <parent link="chassis" />
+    <child link="hokuyo" />
+  </joint>
 </robot>
